Commit message: update base -> base_link

File: b2_description/xacro/gazebo.xacro (robot description, xacro)
@@ -2,5 +2,5 @@
 <robot xmlns:xacro="http://www.ros.org/wiki/xacro" >
     <xacro:macro  name="robot_gazebo_sensors" params="robot_name">
-        <gazebo reference="base">
+        <gazebo reference="base_link">
             <turnGravityOff>false</turnGravityOff>
         </gazebo>

File: b2_description/xacro/robot.xacro (robot description, xacro)
@@ -14,9 +14,9 @@
             <origin rpy="0 0 0" xyz="0 0 0"/>
             <parent link="world"/>
-            <child link="base"/>
+            <child link="base_link"/>
         </joint>
     </xacro:if>
     <joint name='laser_scan' type='fixed'>
-        <parent link="base"/>,
+        <parent link="base_link"/>,
         <child link="laser_frame"/>
         <origin xyz="0.34218 0.0 0.17851" rpy="0 0 0" />
@@ -41,9 +41,9 @@
         </collision>
     </link>
-    <link name="base">
+    <link name="base_link">
     </link>
     <joint name="floating_base" type="fixed">
         <origin rpy="0 0 0" xyz="0 0 0"/>
-        <parent link="base"/>
+        <parent link="base_link"/>
         <child link="trunk"/>
     </joint>
@@ -51,5 +51,5 @@
     </link>
     <joint name="base_footprint_joint" type="fixed">
-        <parent link="base"/>
+        <parent link="base_link"/>
         <child link="base_footprint"/>
         <origin xyz="0 0 0" rpy="0 0 0"/>
@@ -79,5 +79,5 @@
     </link>
     <joint name="imu_joint" type="fixed">
-        <parent link="base"/>
+        <parent link="base_link"/>
         <child link="imu_link"/>
         <origin rpy="0 0 0" xyz="0 0 0"/>
@@ -151,5 +151,5 @@
     </link>
     <joint name="camera_face_joint" type="fixed">
-        <parent link="base"/>
+        <parent link="base_link"/>
         <child link="camera_face"/>
         <origin xyz="0.42 0 0.005" rpy="0 0 0"/>

File: b2w_description/xacro/gazebo.xacro (robot description, xacro)
@@ -2,5 +2,5 @@
 <robot xmlns:xacro="http://www.ros.org/wiki/xacro" >
     <xacro:macro  name="robot_gazebo_sensors" params="robot_name">
-        <gazebo reference="base">
+        <gazebo reference="base_link">
             <turnGravityOff>false</turnGravityOff>
         </gazebo>

File: b2w_description/xacro/robot.xacro (robot description, xacro)
@@ -14,9 +14,9 @@
             <origin rpy="0 0 0" xyz="0 0 0"/>
             <parent link="world"/>
-            <child link="base"/>
+            <child link="base_link"/>
         </joint>
     </xacro:if>
     <joint name='laser_scan' type='fixed'>
-        <parent link="base"/>,
+        <parent link="base_link"/>,
         <child link="laser_frame"/>
         <origin xyz="0.34218 0.0 0.17851" rpy="0 0 0" />
@@ -41,9 +41,9 @@
         </collision>
     </link>
-    <link name="base">
+    <link name="base_link">
     </link>
     <joint name="floating_base" type="fixed">
         <origin rpy="0 0 0" xyz="0 0 0"/>
-        <parent link="base"/>
+        <parent link="base_link"/>
         <child link="trunk"/>
     </joint>
@@ -51,5 +51,5 @@
     </link>
     <joint name="base_footprint_joint" type="fixed">
-        <parent link="base"/>
+        <parent link="base_link"/>
         <child link="base_footprint"/>
         <origin xyz="0 0 0" rpy="0 0 0"/>
@@ -79,5 +79,5 @@
     </link>
     <joint name="imu_joint" type="fixed">
-        <parent link="base"/>
+        <parent link="base_link"/>
         <child link="imu_link"/>
         <origin rpy="0 0 0" xyz="0 0 0"/>
@@ -151,5 +151,5 @@
     </link>
     <joint name="camera_face_joint" type="fixed">
-        <parent link="base"/>
+        <parent link="base_link"/>
         <child link="camera_face"/>
         <origin xyz="0.42 0 0.005" rpy="0 0 0"/>
